File: hw/sch_pcb/TFCO201.kicad_sch (KiCad schematic)
At the start: 19 parts, among them J1 SM04B-GHS-TB, J2 SM04B-GHS-TB, M1 M3, M2 M3, M3 M3, M4 M3, M5 M3, M6 M3, U2 SCD41-D-R2, U3 MIC5504-3.3YM5

Commit message: Update title block.
Other:
- title: TFHT01B -> TFCO201A
Changed lines of the file:
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@@
   (paper "A4")
   (title_block
-    (title "TFHT01B")
-    (date "2021-04-05")
+    (title "TFCO201A")
+    (date "2023-10-01")
     (company "ThunderFly s.r.o.")
-    (comment 1 "UAV Humidity and Temperature \\n sensor \\n ")
+    (comment 1 "UAV CO2 concentration sensor. ")
     (comment 2 "kaklik  <info@thunderfly.cz>")
   )
